File: clackade.kicad_pcb (KiCad board)
At the start: 2 copper layers, 63.3 x 101.1 mm, 13 parts, among them SW1 SW_Push, SW2 SW_Push, SW3 SW_Push, SW4 SW_Push, U1 XIAO-RP2040-DIP

Commit message: Add files via upload
Parts:
- added G***: LOGO, LOGO, F.Cu at (85.2, 101.8)
- added G***: LOGO, LOGO, F.Cu at (86.6, 78.5)
- added G***: LOGO, LOGO, F.Cu at (108.6, 105.5)
- added G***: LOGO, LOGO, F.Cu at (78.4, 148.9)
- added G***: LOGO, LOGO, B.Cu at (114.5, 111.3)
- added G***: LOGO, LOGO, B.Cu at (86.6, 110.3)
- moved U1 42.7 mm to (114.6, 71.7)
- moved SW2 26.8 mm to (81.2, 127.0)
- moved SW1 26.8 mm to (100.4, 117.3)
- moved SW3 26.7 mm to (119.5, 126.8)
- moved SW4 26.7 mm to (100.3, 136.3)
- moved D2 26.4 mm to (85.0, 89.7)
- moved D1 26.4 mm to (97.9, 81.3)
- moved D3 26.4 mm to (111.9, 90.0)
- moved D4 26.4 mm to (97.9, 98.8)
- moved R1 26.4 mm to (75.8, 67.0)
- moved R2 26.4 mm to (83.4, 67.0)
- moved R4 10.5 mm to (98.6, 67.5)
- moved R3 10.3 mm to (91.0, 67.3)
Routing:
- net GND: track 0.00 -> 173.7 mm
- net SW2: track 0.00 -> 96.7 mm, vias 0 -> 1
- net SW4: track 0.00 -> 60.6 mm
- net SW1: track 0.00 -> 58.1 mm, vias 0 -> 1
- net SW3: track 0.00 -> 56.1 mm
- net LED1: track 0.00 -> 49.4 mm
- net LED2: track 0.00 -> 40.7 mm
- net LED3: track 0.00 -> 33.5 mm
- net Net-(D3-PadA): track 0.00 -> 33.5 mm
- net Net-(D4-PadA): track 0.00 -> 32.3 mm
- net Net-(D1-PadA): track 0.00 -> 31.2 mm
- net LED4: track 0.00 -> 26.2 mm
- net Net-(D2-PadA): track 0.00 -> 24.7 mm
- net unconnected-(U1-VBUS-Pad14): track 0.00 -> 0.84 mm
- net unconnected-(U1-GPIO6/SDA-Pad5): track 0.00 -> 0.84 mm
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Other:
- board size 63.3 x 101.1 mm -> 61.3 x 97.9 mm
